Commit message: added comments

File: ros_ws/src/amr/urdf/common_properties.xacro (robot description, xacro)
@@ -1,8 +1,9 @@
 <?xml version="1.0"?>        <!-- to recognize the file as xml file, URDF uses metric system -->
 <robot xmlns:xacro="http://www.ros.org/wiki/xacro">
+    <!-- colour tags -->
     <material name="black">
         <color rgba="0.0 0.0 0.0 1.0"/>
     </material>
-    <material name="blue">  <!-- set colour name-->
+    <material name="blue">
         <color rgba="0 0 0.8 1" />
     </material>
@@ -10,5 +11,5 @@
         <color rgba="0.0 0.8 0.0 1.0"/>
     </material>
-    <material name="grey">  <!-- set colour name-->
+    <material name="grey">
         <color rgba="0.5 0.5 0.5 1" />
     </material>
@@ -28,4 +29,5 @@
         <color rgba="1.0 1.0 1.0 1.0"/>
     </material>
+    <!-- macros for defining inertia -->
     <xacro:macro name="box_inertia" params="m l w h xyz rpy">
         <inertial>

File: ros_ws/src/amr/urdf/lidar.xacro (robot description, xacro)
@@ -1,4 +1,5 @@
 <?xml version="1.0"?>
 <robot xmlns:xacro="http://www.ros.org/wiki/xacro">
+    <!-- laser joint-->
     <joint name="laser_joint" type="fixed" >
         <parent link="base_link" />
@@ -6,4 +7,5 @@
         <origin xyz="0 0 0.035" rpy="0 0 0" />
     </joint>
+    <!-- laser frame -->
     <link name="laser_frame">    <!-- set second link name -->
         <visual>
@@ -23,4 +25,5 @@
                                 xyz="0 0 0" rpy="0 0 0" />
     </link>
+    <!-- laser reference for gazebo -->
     <gazebo reference="laser_frame">
         <material>Gazebo/Red</material>

File: ros_ws/src/amr/urdf/robot_base.xacro (robot description, xacro)
@@ -65,4 +65,5 @@
                                 xyz="0 0 0" rpy="0 0 0" />
     </link>
+    <!-- macro for defining castor wheel links -->
     <xacro:macro name="castor_wheel_link" params="prefix">
         <link name="${prefix}_castor_wheel_link">    <!-- set second link name -->
@@ -89,10 +90,10 @@
     <xacro:castor_wheel_link prefix="front_left" />
     <!-- robot joints -->
-    <joint name="footprint_base_joint" type="fixed">     <!-- set joint name and type-->
+    <joint name="footprint_base_joint" type="fixed">
         <parent link="base_footprint" />
         <child link="base_link" />
         <origin xyz="0 0 ${wheel_radius + 0.097}" rpy="0 0 0" />
     </joint>
-    <joint name="base_right_wheel_joint" type="continuous">     <!-- set joint name and type-->
+    <joint name="base_right_wheel_joint" type="continuous">
         <parent link="base_link" />
         <child link="left_wheel_link" />
@@ -100,5 +101,5 @@
         <axis xyz="0 0 -1" />
     </joint>
-    <joint name="base_left_wheel_joint" type="continuous">     <!-- set joint name and type-->
+    <joint name="base_left_wheel_joint" type="continuous">
         <parent link="base_link" />
         <child link="right_wheel_link" />
@@ -106,6 +107,7 @@
         <axis xyz="0 0 -1" />
     </joint>
+    <!-- macro for defining castor wheel joints -->
     <xacro:macro name="castor_wheel_joint" params="prefix parent child xyz rpy axis">
-        <joint name="${prefix}_joint" type="fixed">     <!-- set joint name and type-->
+        <joint name="${prefix}_joint" type="fixed">
             <parent link="${parent}" />
             <child link="${child}" />

File: ros_ws/src/amr/urdf/robot_base_gazebo.xacro (robot description, xacro)
@@ -1,33 +1,35 @@
 <?xml version="1.0"?>
 <robot xmlns:xacro="http://www.ros.org/wiki/xacro">
-    <gazebo reference="base_link" >          <!-- gazebo refernce in this tag is for specific to that link-->
+    <!-- gazebo reference tags for links -->
+    <gazebo reference="base_link" >
         <material> Gazebo/Blue </material>
     </gazebo>
-    <gazebo reference="right_wheel_link" >          <!-- gazebo refernce in this tag is for specific to that link-->
+    <gazebo reference="right_wheel_link" >
         <material> Gazebo/Grey </material>
     </gazebo>
-    <gazebo reference="left_wheel_link" >          <!-- gazebo refernce in this tag is for specific to that link-->
+    <gazebo reference="left_wheel_link" >
         <material> Gazebo/Grey </material>
     </gazebo>
-    <gazebo reference="front_right_castor_wheel_link" >          <!-- gazebo refernce in this tag is for specific to that link-->
+    <gazebo reference="front_right_castor_wheel_link" >
         <material> Gazebo/Grey </material>
         <mu1 value="0.01" />
         <mu2 value="0.01" />
     </gazebo>
-    <gazebo reference="back_right_castor_wheel_link" >          <!-- gazebo refernce in this tag is for specific to that link-->
+    <gazebo reference="back_right_castor_wheel_link" >
         <material> Gazebo/Grey </material>
         <mu1 value="0.01" />
         <mu2 value="0.01" />
     </gazebo>
-    <gazebo reference="back_left_castor_wheel_link" >          <!-- gazebo refernce in this tag is for specific to that link-->
+    <gazebo reference="back_left_castor_wheel_link" >
         <material> Gazebo/Grey </material>
         <mu1 value="0.01" />
         <mu2 value="0.01" />
     </gazebo>
-    <gazebo reference="front_left_castor_wheel_link" >          <!-- gazebo refernce in this tag is for specific to that link-->
+    <gazebo reference="front_left_castor_wheel_link" >
         <material> Gazebo/Grey </material>
         <mu1 value="0.01" />
         <mu2 value="0.01" />
     </gazebo>
+    <!-- gazebo reference for differential drive(amr) -->
     <gazebo>
         <plugin name="diff_drive_controller" filename="libgazebo_ros_diff_drive.so">
