Commit message: changes according to gazebo harmonic

File: ros_ws/src/amr/urdf/lidar.xacro (robot description, xacro)
@@ -45,5 +45,5 @@
                 </range>
             </ray>
-            <plugin name="laser_controller" filename="libgazebo_ros_ray_sensor.so">
+            <!-- <plugin name="laser_controller" filename="libgazebo_ros_ray_sensor.so">
                 <ros>
                     <remapping>~/out:=scan</remapping>
@@ -51,5 +51,5 @@
                 <output_type>sensor_msgs/LaserScan</output_type>
                 <frame_name>laser_frame</frame_name>
-            </plugin>
+            </plugin> -->
         </sensor>
     </gazebo>

File: ros_ws/src/amr/urdf/robot.xacro (robot description, xacro)
@@ -4,4 +4,4 @@
     <xacro:include filename="robot_base.xacro" />
     <xacro:include filename="robot_base_gazebo.xacro" />
-    <xacro:include filename="lidar.xacro" />
+    <!-- <xacro:include filename="lidar.xacro" /> -->
 </robot>

File: ros_ws/src/amr/urdf/robot_base.xacro (robot description, xacro)
@@ -16,6 +16,6 @@
         <visual>
             <geometry>
-                <!-- <box size="${base_length} ${base_width} ${base_height}" /> -->
-                <mesh filename="package://amr/meshes/base_link.stl" scale="0.001 0.001 0.001" />
+                <box size="${base_length} ${base_width} ${base_height}" />
+                <!-- <mesh filename="package://amr/meshes/base_link.stl" scale="0.001 0.001 0.001" /> -->
             </geometry>
             <origin xyz="0 0 0" rpy="0 0 0" />
@@ -37,5 +37,5 @@
             </geometry>
             <origin xyz="0 0 0" rpy="0 0 0" />
-            <material name="grey" />
+            <material name="red" />
         </visual>
         <collision>
@@ -54,5 +54,5 @@
             </geometry>
             <origin xyz="0 0 0" rpy="0 0 0" />
-            <material name="grey" />
+            <material name="red" />
         </visual>
         <collision>

File: ros_ws/src/amr/urdf/robot_base_gazebo.xacro (robot description, xacro)
@@ -1,39 +1,35 @@
 <?xml version="1.0"?>
 <robot xmlns:xacro="http://www.ros.org/wiki/xacro">
-    <!-- gazebo reference tags for links -->
-    <gazebo reference="base_link" >
+    <gazebo reference="base_link" >          <!-- gazebo refernce in this tag is for specific to that link-->
         <material> Gazebo/Blue </material>
     </gazebo>
-    <gazebo reference="right_wheel_link" >
+    <gazebo reference="right_wheel_link" >          <!-- gazebo refernce in this tag is for specific to that link-->
+        <material> Gazebo/Red </material>
+    </gazebo>
+    <gazebo reference="left_wheel_link" >          <!-- gazebo refernce in this tag is for specific to that link-->
+        <material> Gazebo/Red </material>
+    </gazebo>
+    <gazebo reference="front_right_castor_wheel_link" >          <!-- gazebo refernce in this tag is for specific to that link-->
         <material> Gazebo/Grey </material>
+        <mu1 value="0.1" />
+        <mu2 value="0.1" />
     </gazebo>
-    <gazebo reference="left_wheel_link" >
+    <gazebo reference="back_right_castor_wheel_link" >          <!-- gazebo refernce in this tag is for specific to that link-->
         <material> Gazebo/Grey </material>
+        <mu1 value="0.1" />
+        <mu2 value="0.1" />
     </gazebo>
-    <gazebo reference="front_right_castor_wheel_link" >
+    <gazebo reference="back_left_castor_wheel_link" >          <!-- gazebo refernce in this tag is for specific to that link-->
         <material> Gazebo/Grey </material>
-        <mu1 value="0.01" />
-        <mu2 value="0.01" />
+        <mu1 value="0.1" />
+        <mu2 value="0.1" />
     </gazebo>
-    <gazebo reference="back_right_castor_wheel_link" >
+    <gazebo reference="front_left_castor_wheel_link" >          <!-- gazebo refernce in this tag is for specific to that link-->
         <material> Gazebo/Grey </material>
-        <mu1 value="0.01" />
-        <mu2 value="0.01" />
+        <mu1 value="0.1" />
+        <mu2 value="0.1" />
     </gazebo>
-    <gazebo reference="back_left_castor_wheel_link" >
-        <material> Gazebo/Grey </material>
-        <mu1 value="0.01" />
-        <mu2 value="0.01" />
-    </gazebo>
-    <gazebo reference="front_left_castor_wheel_link" >
-        <material> Gazebo/Grey </material>
-        <mu1 value="0.01" />
-        <mu2 value="0.01" />
-    </gazebo>
-    <!-- gazebo reference for differential drive(amr) -->
     <gazebo>
-        <plugin name="diff_drive_controller" filename="libgazebo_ros_diff_drive.so">
-        <!-- Update rate in Hz -->
-        <update_rate>50</update_rate>   <!--rate to update position-->
+        <plugin filename="gz-sim-diff-drive-system" name="gz::sim::systems::DiffDrive">
         <!-- wheels -->
         <left_joint>base_left_wheel_joint</left_joint>
@@ -41,18 +37,15 @@
         <!-- kinematics -->
         <wheel_separation>0.45</wheel_separation>
-        <wheel_diameter>0.2</wheel_diameter>
-        <!-- limits -->
-        <max_wheel_torque>20</max_wheel_torque>
-        <max_wheel_acceleration>1.0</max_wheel_acceleration>
-        <!-- input -->
-        <command_topic>cmd_vel</command_topic>
-        <!-- output -->
-        <publish_odom>true</publish_odom>
-        <publish_odom_tf>true</publish_odom_tf>
-        <publish_wheel_tf>true</publish_wheel_tf>
-        <odometry_topic>odom</odometry_topic>
-        <odometry_frame>odom</odometry_frame>
-        <robot_base_frame>base_footprint</robot_base_frame>
+        <wheel_radius>0.2</wheel_radius>
+        <frame_id>odom</frame_id>
+        <child_frame_id>base_footprint</child_frame_id>
         </plugin>
     </gazebo>
+    <gazebo>
+        <plugin
+            filename="gz-sim-joint-state-publisher-system" name="gz::sim::systems::JointStatePublisher">
+            <left_joint>base_left_wheel_joint</left_joint>
+            <right_joint>base_right_wheel_joint</right_joint>
+    </plugin>
+    </gazebo>
 </robot>

Commit message: changes

File: ros_ws/src/amr/urdf/lidar.xacro (robot description, xacro)
@@ -5,5 +5,5 @@
         <parent link="base_link" />
         <child link="laser_frame" />
-        <origin xyz="0 0 0.035" rpy="0 0 0" />
+        <origin xyz="0.22 0 0.035" rpy="0 0 0" />
     </joint>
     <!-- laser frame -->

File: ros_ws/src/amr/urdf/ros2_control.xacro (robot description, xacro)
@@ -6,6 +6,6 @@
         <param name="left_wheel_name">base_left_wheel_joint</param>
         <param name="right_wheel_name">base_right_wheel_joint</param>
-        <param name="enc_counts_per_rev">8192</param>
-        <param name="wheel_separation">0.10</param>
+        <param name="enc_counts_per_rev">2392</param>
+        <param name="wheel_separation">0.54</param>
         <param name="pid_p">20</param>
         <param name="pid_d">12</param>

Commit message: changes

File: ros_ws/src/amr/urdf/lidar.xacro (robot description, xacro)
@@ -5,5 +5,5 @@
         <parent link="base_link" />
         <child link="laser_frame" />
-        <origin xyz="0.22 0 0.035" rpy="0 0 0" />
+        <origin xyz="0.22 0 0.035" rpy="0 0 ${pi}" />
     </joint>
     <!-- laser frame -->

File: ros_ws/src/amr/urdf/robot_base.xacro (robot description, xacro)
@@ -90,5 +90,5 @@
     <xacro:castor_wheel_link prefix="front_left" />
     <!-- robot joints -->
-    <joint name="footprint_base_joint" type="fixed">
+    <joint name="footprint_base_jont" type="fixed">
         <parent link="base_footprint" />
         <child link="base_link" />

Commit message: changed orientation of lidar sensor

File: ros_ws/src/amr/urdf/lidar.xacro (robot description, xacro)
@@ -5,5 +5,5 @@
         <parent link="base_link" />
         <child link="laser_frame" />
-        <origin xyz="0.22 0 0.035" rpy="0 0 ${pi}" />
+        <origin xyz="0.22 0 0.035" rpy="0 0 0" />
     </joint>
     <!-- laser frame -->
