Commit message: changes

File: ros_ws/src/amr/urdf/robot.xacro (robot description, xacro)
@@ -1,8 +1,13 @@
 <?xml version="1.0"?>
 <robot name="amr" xmlns:xacro="http://www.ros.org/wiki/xacro">
+    <xacro:arg name="use_ros2_control" default="true" />
     <xacro:include filename="common_properties.xacro" />
     <xacro:include filename="robot_base.xacro" />
-    <!-- <xacro:include filename="robot_base_gazebo.xacro" /> -->
-    <xacro:include filename="ros2_control.xacro" />
+    <xacro:if value="$(arg use_ros2_control)">
+        <xacro:include filename="ros2_control.xacro" />
+    </xacro:if>
+    <xacro:unless value="$(arg use_ros2_control)">
+        <xacro:include filename="robot_base_gazebo.xacro" />
+    </xacro:unless>
     <xacro:include filename="lidar.xacro" />
 </robot>

File: ros_ws/src/amr/urdf/robot_base_gazebo.xacro (robot description, xacro)
@@ -5,8 +5,8 @@
     </gazebo>
     <gazebo reference="right_wheel_link" >          <!-- gazebo refernce in this tag is for specific to that link-->
-        <material> Gazebo/Red </material>
+        <material> Gazebo/Blue </material>
     </gazebo>
     <gazebo reference="left_wheel_link" >          <!-- gazebo refernce in this tag is for specific to that link-->
-        <material> Gazebo/Red </material>
+        <material> Gazebo/Blue </material>
     </gazebo>
     <gazebo reference="front_right_castor_wheel_link" >          <!-- gazebo refernce in this tag is for specific to that link-->
@@ -36,5 +36,5 @@
         <right_joint>base_right_wheel_joint</right_joint>
         <!-- kinematics -->
-        <wheel_separation>0.45</wheel_separation>
+        <wheel_separation>0.54</wheel_separation>
         <wheel_radius>0.2</wheel_radius>
         <frame_id>odom</frame_id>

File: ros_ws/src/amr/urdf/ros2_control.xacro (robot description, xacro)
@@ -1,5 +1,80 @@
 <?xml version="1.0"?>        <!-- to recognize the file as xml file, URDF uses metric system -->
 <robot xmlns:xacro="http://www.ros.org/wiki/xacro">
-    <ros2_control name="RealRobot" type="system">
+    <xacro:arg name="use_ros2_control" default="true" />
+    <xacro:if value="$(arg use_ros2_control)">
+        <ros2_control name="RealRobot" type="system">
+            <hardware>
+                <plugin>diff_drive/DiffDriveHardware</plugin>
+                <param name="left_wheel_name">base_left_wheel_joint</param>
+                <param name="right_wheel_name">base_right_wheel_joint</param>
+                <param name="enc_counts_per_rev_l">2329</param>
+                <param name="enc_counts_per_rev_r">2376</param>
+                <param name="wheel_separation">0.54</param>
+                <param name="pid_p">20</param>
+                <param name="pid_d">12</param>
+                <param name="pid_i">0</param>
+                <param name="pid_o">50</param>
+            </hardware>
+            <joint name="base_left_wheel_joint">
+                <command_interface name="velocity"/>
+                <state_interface name="position"/>
+                <state_interface name="velocity"/>
+            </joint>
+            <joint name="base_right_wheel_joint">
+                <command_interface name="velocity"/>
+                <state_interface name="position"/>
+                <state_interface name="velocity"/>
+            </joint>
+        </ros2_control>
+    </xacro:if>
+    <xacro:unless value="$(arg use_ros2_control)">
+        <ros2_control name="GazeboSimSystem" type="system">
+            <hardware>
+                <plugin>gz_ros2_control/GazeboSimSystem</plugin>
+            </hardware>
+            <joint name="base_left_wheel_joint">
+                <command_interface name="velocity">
+                    <param name="min">-10</param>
+                    <param name="max">10</param>
+                </command_interface>
+                <state_interface name="position"/>
+                <state_interface name="velocity"/>
+            </joint>
+            <joint name="base_right_wheel_joint">
+                <command_interface name="velocity">
+                    <param name="min">-10</param>
+                    <param name="max">10</param>
+                </command_interface>
+                <state_interface name="position"/>
+                <state_interface name="velocity"/>
+            </joint>
+        </ros2_control>
+        <gazebo>
+            <plugin filename="gz_ros2_control-system" name="gz_ros2_control::GazeboSimROS2ControlPlugin">
+                <parameters>$(find amr)/config/controllers.yaml</parameters>
+            </plugin>
+        </gazebo>
+        <gazebo reference="front_right_castor_wheel_link" >          <!-- gazebo refernce in this tag is for specific to that link-->
+            <material> Gazebo/Grey </material>
+            <mu1 value="0.1" />
+            <mu2 value="0.1" />
+        </gazebo>
+        <gazebo reference="back_right_castor_wheel_link" >          <!-- gazebo refernce in this tag is for specific to that link-->
+            <material> Gazebo/Grey </material>
+            <mu1 value="0.1" />
+            <mu2 value="0.1" />
+        </gazebo>
+        <gazebo reference="back_left_castor_wheel_link" >          <!-- gazebo refernce in this tag is for specific to that link-->
+            <material> Gazebo/Grey </material>
+            <mu1 value="0.1" />
+            <mu2 value="0.1" />
+        </gazebo>
+        <gazebo reference="front_left_castor_wheel_link" >          <!-- gazebo refernce in this tag is for specific to that link-->
+            <material> Gazebo/Grey </material>
+            <mu1 value="0.1" />
+            <mu2 value="0.1" />
+        </gazebo>
+    </xacro:unless>
+    <!-- <ros2_control name="RealRobot" type="system">
       <hardware>
         <plugin>diff_drive/DiffDriveHardware</plugin>
@@ -25,5 +100,5 @@
       </joint>
     </ros2_control>
-    <!-- <ros2_control name="GazeboSimSystem" type="system">
+    <ros2_control name="GazeboSimSystem" type="system">
         <hardware>
             <plugin>gz_ros2_control/GazeboSimSystem</plugin>
@@ -45,10 +120,29 @@
             <state_interface name="velocity"/>
         </joint>
-    </ros2_control> -->
+    </ros2_control>
     <gazebo>
-        <!-- Joint state publisher -->
         <plugin filename="gz_ros2_control-system" name="gz_ros2_control::GazeboSimROS2ControlPlugin">
             <parameters>$(find amr)/config/controllers.yaml</parameters>
         </plugin>
     </gazebo>
+        <gazebo reference="front_right_castor_wheel_link" >
+        <material> Gazebo/Grey </material>
+        <mu1 value="0.1" />
+        <mu2 value="0.1" />
+    </gazebo>
+    <gazebo reference="back_right_castor_wheel_link" >
+        <material> Gazebo/Grey </material>
+        <mu1 value="0.1" />
+        <mu2 value="0.1" />
+    </gazebo>
+    <gazebo reference="back_left_castor_wheel_link" >
+        <material> Gazebo/Grey </material>
+        <mu1 value="0.1" />
+        <mu2 value="0.1" />
+    </gazebo>
+    <gazebo reference="front_left_castor_wheel_link" >
+        <material> Gazebo/Grey </material>
+        <mu1 value="0.1" />
+        <mu2 value="0.1" />
+    </gazebo> -->
 </robot>
