Commit message: updated position of sensor

File: ros_ws/src/amr/urdf/ultrasonic.xacro (robot description, xacro)
@@ -8,5 +8,5 @@
         <parent link="base_link" />
         <child link="ultrasonic_sensor" />
-        <origin xyz="${0.3 - ultrasonic_radius} ${0.25 - ultrasonic_length} 0.0275" rpy="${pi/2} 0 ${pi / 4}" />
+        <origin xyz="${0.3 - ultrasonic_radius} ${0.25 - ultrasonic_length} 0.0275" rpy="0 0 0" />
     </joint>
     <link name="ultrasonic_sensor">
@@ -15,5 +15,5 @@
                 <cylinder radius="${ultrasonic_radius}" length="${ultrasonic_length}"/>
             </geometry>
-            <origin xyz="0 0 0" rpy="0 0 0"/>
+            <origin xyz="0 0 0" rpy="${pi / 2} 0 0"/>
             <material name="green"/>
         </visual>
