Commit message: left and right wheel name correction

File: ros_ws/src/amr/urdf/robot_base.xacro (robot description, xacro)
@@ -31,5 +31,5 @@
                            xyz="0 0 ${wheel_radius}" rpy="0 0 0" />
     </link>
-    <link name="right_wheel_link">    <!-- set second link name -->
+    <link name="left_wheel_link">    <!-- set second link name -->
         <visual>
             <geometry>
@@ -48,5 +48,5 @@
                                 xyz="0 0 0" rpy="0 0 0" />
     </link>
-    <link name="left_wheel_link">    <!-- set second link name -->
+    <link name="right_wheel_link">    <!-- set second link name -->
         <visual>
             <geometry>
@@ -97,5 +97,5 @@
     <joint name="base_right_wheel_joint" type="continuous">
         <parent link="base_link" />
-        <child link="left_wheel_link" />
+        <child link="right_wheel_link" />
         <origin xyz="0 -0.27 -0.097" rpy="${pi / 2} 0 0" />
         <axis xyz="0 0 -1" />
@@ -103,5 +103,5 @@
     <joint name="base_left_wheel_joint" type="continuous">
         <parent link="base_link" />
-        <child link="right_wheel_link" />
+        <child link="left_wheel_link" />
         <origin xyz="0 0.27 -0.097" rpy="${pi / 2} 0 0" />
         <axis xyz="0 0 -1" />
